File: kicad/SC08v2.kicad_pcb (KiCad board)
At the start: 2 copper layers, 23 parts, among them U17 74HC86, U18 74HC86, U19 74HC00, U20 74HC00, U21 74HC85, U22 74HC85, U23 74HC283, U24 74HC151, U25 74HC151, U26 74HC283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

Commit message: kicad: finalize sketch
Parts:
- removed AUX_0, DTA1, DTB1, INP0, IR1, OUT1: 74HC273, Package_DIP:DIP-20_W7.62mm
- removed U17, U18: 74HC86, Package_DIP:DIP-14_W7.62mm
- removed U19, U20: 74HC00, Package_DIP:DIP-14_W7.62mm
- removed U21, U22: 74HC85, Package_DIP:DIP-16_W7.62mm
- removed U23, U26: 74HC283, Package_DIP:DIP-16_W7.62mm
- removed U24, U25, U27, U28, U29, U30, U31, U32: 74HC151, Package_DIP:DIP-16_W7.62mm
- removed U5: LM555xN, Package_DIP:DIP-8_W7.62mm
Other:
- copper layers 2 -> 4
