File: kicad/alu.kicad_sch (KiCad schematic)
At the start: 32 parts, among them U17 74HC86, U18 74HC86, U19 74HC00, U20 74HC00, U21 74HC85, U22 74HC85, U23 74HC283, U24 74HC151, U25 74HC151, U26 74HC283, U27 74HC151, U28 74HC151, U29 74HC151, U30 74HC151, U31 74HC151, U32 74HC151

Commit message: kicad: compact design
Other:
- note added: "ADD INPUT INVERTER"
- note added: "ADDITION"
- note added: "BITWISE NAND"
- note added: "COMPARATION"
- note added: "MULTIPLEXED OUTPUT"
- note removed: "ADDER"
- note removed: "COMPARATOR"
- note removed: "INVERTER"
- note removed: "MULTIPLEXER"
- note removed: "NAND"
- moved on the sheet: C12, C13, C14, C15, C16, C17, C18, C19, C20, C21, C22, C23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

Commit message: kicad: finalize sketch
Parts:
- ADD_U0_C1: renamed from C51; footprint (none) -> Capacitor_THT:C_Disc_D3.0mm_W1.6mm_P2.50mm
- ADD_U1_C1: renamed from C52; footprint (none) -> Capacitor_THT:C_Disc_D3.0mm_W1.6mm_P2.50mm
- ALUMUX_U0_C1: renamed from C12; footprint (none) -> Capacitor_THT:C_Disc_D3.0mm_W1.6mm_P2.50mm
- ALUMUX_U1_C1: renamed from C13; footprint (none) -> Capacitor_THT:C_Disc_D3.0mm_W1.6mm_P2.50mm
- ALUMUX_U2_C1: renamed from C19; footprint (none) -> Capacitor_THT:C_Disc_D3.0mm_W1.6mm_P2.50mm
- ALUMUX_U3_C1: renamed from C18; footprint (none) -> Capacitor_THT:C_Disc_D3.0mm_W1.6mm_P2.50mm
- ALUMUX_U4_C1: renamed from C14; footprint (none) -> Capacitor_THT:C_Disc_D3.0mm_W1.6mm_P2.50mm
- ALUMUX_U5_C1: renamed from C15; footprint (none) -> Capacitor_THT:C_Disc_D3.0mm_W1.6mm_P2.50mm
- ALUMUX_U6_C1: renamed from C16; footprint (none) -> Capacitor_THT:C_Disc_D3.0mm_W1.6mm_P2.50mm
- ALUMUX_U7_C1: renamed from C17; footprint (none) -> Capacitor_THT:C_Disc_D3.0mm_W1.6mm_P2.50mm
- COMP_U0_C1: renamed from C24; footprint (none) -> Capacitor_THT:C_Disc_D3.0mm_W1.6mm_P2.50mm
- COMP_U0_C2: renamed from C25; footprint (none) -> Capacitor_THT:C_Disc_D3.0mm_W1.6mm_P2.50mm
- NAND_U0_C1: renamed from C22; footprint (none) -> Capacitor_THT:C_Disc_D3.0mm_W1.6mm_P2.50mm
- NAND_U1_C1: renamed from C23; footprint (none) -> Capacitor_THT:C_Disc_D3.0mm_W1.6mm_P2.50mm
- XOR_U0_C1: renamed from C20; footprint (none) -> Capacitor_THT:C_Disc_D3.0mm_W1.6mm_P2.50mm
- XOR_U1_C1: renamed from C21; footprint (none) -> Capacitor_THT:C_Disc_D3.0mm_W1.6mm_P2.50mm
- renumbered U23 to ADD_U0, U26 to ADD_U1, U24 to ALUMUX_U0, U27 to ALUMUX_U1, U29 to ALUMUX_U2, U31 to ALUMUX_U3, U25 to ALUMUX_U4, U28 to ALUMUX_U5, U30 to ALUMUX_U6, U32 to ALUMUX_U7, U21 to COMP_U0, U22 to COMP_U1, U19 to NAND_U0, U20 to NAND_U1, U17 to XOR_U0, U18 to XOR_U1
Connections:
- no-connect marks 0 -> 9
