File: kicad/clk.kicad_sch (KiCad schematic)
At the start: 7 parts, among them U43 74HC04, U5 LM555xN

Commit message: kicad: finalize sketch
Parts:
- CLKINVERTER_U1: renamed from U43; footprint (none) -> Package_DIP:DIP-14_W7.62mm
- CLKINVERTER_U_C1: renamed from C27; footprint (none) -> Capacitor_THT:C_Disc_D3.0mm_W1.6mm_P2.50mm
- CLK_U_C1: renamed from C3; footprint (none) -> Capacitor_THT:C_Disc_D3.0mm_W1.6mm_P2.50mm
- CLK_U_C2: renamed from C26; footprint (none) -> Capacitor_THT:C_Disc_D3.0mm_W1.6mm_P2.50mm
- CLK_U_C3: renamed from C4; footprint (none) -> Capacitor_THT:C_Disc_D3.0mm_W1.6mm_P2.50mm
- CLK_U_R1: renamed from R2; footprint (none) -> Resistor_THT:R_Axial_DIN0204_L3.6mm_D1.6mm_P5.08mm_Horizontal
- renumbered U5 to CLK_U1
Connections:
- no-connect marks 0 -> 11
Changed lines of the file:
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@@
 		(color 0 0 0 0)
+	)
+	(no_connect
+		(at 63.5 38.1)
+	)
+	(no_connect
+		(at 172.72 62.23)
+	)
+	(no_connect
+		(at 172.72 77.47)
+	)
+	(no_connect
+		(at 187.96 77.47)
+	)
+	(no_connect
+		(at 187.96 48.26)
+	)
+	(no_connect
+		(at 172.72 33.02)
+	)
+	(no_connect
+		(at 172.72 48.26)
+	)
+	(no_connect
+		(at 187.96 62.23)
+	)
+	(no_connect
+		(at 172.72 91.44)
+	)
+	(no_connect
+		(at 187.96 91.44)
+	)
+	(no_connect
+		(at 187.96 33.02)
 	)
 	(wire
@@
 		(dnp no)
 		(fields_autoplaced yes)
-		(property "Reference" "U43"
+		(property "Reference" "CLKINVERTER_U1"
 			(at 86.36 24.13 0)
 			(effects
@@
 			)
 		)
-		(property "Footprint" ""
+		(property "Footprint" "Package_DIP:DIP-14_W7.62mm"
 			(at 86.36 33.02 0)
 			(effects
@@
 			(project "SC08v2"
 				(path "/8273a279-6d4f-43cc-a94b-c590a7d8a356/48e73f4a-0468-4785-880e-8771bf9b7a5f"
-					(reference "U43")
+					(reference "CLKINVERTER_U1")
 					(unit 1)
 				)
@@
 		(dnp no)
 		(fields_autoplaced yes)
-		(property "Reference" "U43"
+		(property "Reference" "CLKINVERTER_U1"
 			(at 92.71 66.0399 0)
 			(effects
@@
 			)
 		)
-		(property "Footprint" ""
+		(property "Footprint" "Package_DIP:DIP-14_W7.62mm"
 			(at 86.36 67.31 0)
 			(effects
@@
 			(project "SC08v2"
 				(path "/8273a279-6d4f-43cc-a94b-c590a7d8a356/48e73f4a-0468-4785-880e-8771bf9b7a5f"
-					(reference "U43")
+					(reference "CLKINVERTER_U1")
 					(unit 7)
 				)
@@
 		(dnp no)
 		(fields_autoplaced yes)
-		(property "Reference" "U43"
+		(property "Reference" "CLKINVERTER_U1"
 			(at 180.34 24.13 0)
 			(effects
@@
 			)
 		)
-		(property "Footprint" ""
+		(property "Footprint" "Package_DIP:DIP-14_W7.62mm"
 			(at 180.34 33.02 0)
 			(effects
@@
 			(project "SC08v2"
 				(path "/8273a279-6d4f-43cc-a94b-c590a7d8a356/48e73f4a-0468-4785-880e-8771bf9b7a5f"
-					(reference "U43")
+					(reference "CLKINVERTER_U1")
 					(unit 2)
 				)
@@
 		(dnp no)
 		(fields_autoplaced yes)
-		(property "Reference" "U43"
+		(property "Reference" "CLKINVERTER_U1"
 			(at 180.34 39.37 0)
 			(effects
@@
 			)
 		)
-		(property "Footprint" ""
+		(property "Footprint" "Package_DIP:DIP-14_W7.62mm"
 			(at 180.34 48.26 0)
 			(effects
@@
 			(project "SC08v2"
 				(path "/8273a279-6d4f-43cc-a94b-c590a7d8a356/48e73f4a-0468-4785-880e-8771bf9b7a5f"
-					(reference "U43")
+					(reference "CLKINVERTER_U1")
 					(unit 3)
 				)
@@
 		(on_board yes)
 		(dnp no)
-		(property "Reference" "U5"
+		(property "Reference" "CLK_U1"
 			(at 49.276 36.83 0)
 			(effects
@@
 			(project "SC08v2"
 				(path "/8273a279-6d4f-43cc-a94b-c590a7d8a356/48e73f4a-0468-4785-880e-8771bf9b7a5f"
-					(reference "U5")
+					(reference "CLK_U1")
 					(unit 1)
 				)
@@
 		(on_board yes)
 		(dnp no)
-		(property "Reference" "C3"
-			(at 28.194 39.624 0)
+		(property "Reference" "CLK_U_C1"
+			(at 23.114 39.116 0)
 			(effects
 				(font
@@
 			)
 		)
-		(property "Footprint" ""
+		(property "Footprint" "Capacitor_THT:C_Disc_D3.0mm_W1.6mm_P2.50mm"
 			(at 33.9852 45.72 0)
 			(effects
@@
 			(project "SC08v2"
 				(path "/8273a279-6d4f-43cc-a94b-c590a7d8a356/48e73f4a-0468-4785-880e-8771bf9b7a5f"
-					(reference "C3")
+					(reference "CLK_U_C1")
 					(unit 1)
 				)
@@
 		(on_board yes)
 		(dnp no)
-		(property "Reference" "C26"
+		(property "Reference" "CLK_U_C2"
 			(at 58.42 19.304 90)
 			(effects
@@
 			)
 		)
-		(property "Footprint" ""
+		(property "Footprint" "Capacitor_THT:C_Disc_D3.0mm_W1.6mm_P2.50mm"
 			(at 58.42 24.4348 0)
 			(effects
@@
 			(project "SC08v2"
 				(path "/8273a279-6d4f-43cc-a94b-c590a7d8a356/48e73f4a-0468-4785-880e-8771bf9b7a5f"
-					(reference "C26")
+					(reference "CLK_U_C2")
 					(unit 1)
 				)
@@
 		(dnp no)
 		(fields_autoplaced yes)
-		(property "Reference" "U43"
+		(property "Reference" "CLKINVERTER_U1"
 			(at 180.34 68.58 0)
 			(effects
@@
 			)
 		)
-		(property "Footprint" ""
+		(property "Footprint" "Package_DIP:DIP-14_W7.62mm"
 			(at 180.34 77.47 0)
 			(effects
@@
 			(project "SC08v2"
 				(path "/8273a279-6d4f-43cc-a94b-c590a7d8a356/48e73f4a-0468-4785-880e-8771bf9b7a5f"
-					(reference "U43")
+					(reference "CLKINVERTER_U1")
 					(unit 5)
 				)
@@
 		(on_board yes)
 		(dnp no)
-		(property "Reference" "C27"
-			(at 93.98 48.514 90)
+		(property "Reference" "CLKINVERTER_U_C1"
+			(at 98.044 48.514 90)
 			(effects
 				(font
@@
 			)
 		)
-		(property "Footprint" ""
+		(property "Footprint" "Capacitor_THT:C_Disc_D3.0mm_W1.6mm_P2.50mm"
 			(at 93.98 53.6448 0)
 			(effects
@@
 			(project "SC08v2"
 				(path "/8273a279-6d4f-43cc-a94b-c590a7d8a356/48e73f4a-0468-4785-880e-8771bf9b7a5f"
-					(reference "C27")
+					(reference "CLKINVERTER_U_C1")
 					(unit 1)
 				)
@@
 		(dnp no)
 		(fields_autoplaced yes)
-		(property "Reference" "U43"
+		(property "Reference" "CLKINVERTER_U1"
 			(at 180.34 53.34 0)
 			(effects
@@
 			)
 		)
-		(property "Footprint" ""
+		(property "Footprint" "Package_DIP:DIP-14_W7.62mm"
 			(at 180.34 62.23 0)
 			(effects
@@
 			(project "SC08v2"
 				(path "/8273a279-6d4f-43cc-a94b-c590a7d8a356/48e73f4a-0468-4785-880e-8771bf9b7a5f"
-					(reference "U43")
+					(reference "CLKINVERTER_U1")
 					(unit 4)
 				)
@@
 		(dnp no)
 		(fields_autoplaced yes)
-		(property "Reference" "U43"
+		(property "Reference" "CLKINVERTER_U1"
 			(at 180.34 82.55 0)
 			(effects
@@
 			)
 		)
-		(property "Footprint" ""
+		(property "Footprint" "Package_DIP:DIP-14_W7.62mm"
 			(at 180.34 91.44 0)
 			(effects
@@
 			(project "SC08v2"
 				(path "/8273a279-6d4f-43cc-a94b-c590a7d8a356/48e73f4a-0468-4785-880e-8771bf9b7a5f"
-					(reference "U43")
+					(reference "CLKINVERTER_U1")
 					(unit 6)
 				)
@@
 		(dnp no)
 		(fields_autoplaced yes)
-		(property "Reference" "C4"
+		(property "Reference" "CLK_U_C3"
 			(at 67.31 58.4199 0)
 			(effects
@@
 			)
 		)
-		(property "Footprint" ""
+		(property "Footprint" "Capacitor_THT:C_Disc_D3.0mm_W1.6mm_P2.50mm"
 			(at 64.4652 63.5 0)
 			(effects
@@
 			(project "SC08v2"
 				(path "/8273a279-6d4f-43cc-a94b-c590a7d8a356/48e73f4a-0468-4785-880e-8771bf9b7a5f"
-					(reference "C4")
+					(reference "CLK_U_C3")
 					(unit 1)
 				)
@@
 		(dnp no)
 		(fields_autoplaced yes)
-		(property "Reference" "R2"
+		(property "Reference" "CLK_U_R1"
 			(at 29.21 25.3999 0)
 			(effects
@@
 			)
 		)
-		(property "Footprint" ""
+		(property "Footprint" "Resistor_THT:R_Axial_DIN0204_L3.6mm_D1.6mm_P5.08mm_Horizontal"
 			(at 24.892 26.67 90)
 			(effects
@@
 			(project "SC08v2"
 				(path "/8273a279-6d4f-43cc-a94b-c590a7d8a356/48e73f4a-0468-4785-880e-8771bf9b7a5f"
-					(reference "R2")
+					(reference "CLK_U_R1")
 					(unit 1)
 				)
