File: kicad/SC08v2/rom.kicad_sch (KiCad schematic)
At the start: 28 parts

Commit message: Improve and fix docs
Parts:
- ADR1_U0, ADR1_U1, ADR2_U0, ADR2_U1, PC_U0, PC_U1, PC_U2, PC_U3, ROMMUX_U0, ROMMUX_U1, ROMMUX_U2, ROMMUX_U3: value ~ -> (none)
