File: kicad/SC08v2/SC08v2.kicad_pcb (KiCad board)
At the start: 4 copper layers, 0 parts

Commit message: Improve docs and schemas
Parts:
- added ADD_U0: 74HC283, Package_DIP:DIP-16_W7.62mm, F.Cu at (17.6, 16.5)
- added ADD_U0_C1: 100 nF, Capacitor_THT:C_Disc_D3.0mm_W1.6mm_P2.50mm, F.Cu at (60.7, 37.9)
- added ADD_U1: 74HC283, Package_DIP:DIP-16_W7.62mm, F.Cu at (28.4, 16.5)
- added ADD_U1_C1: 100 nF, Capacitor_THT:C_Disc_D3.0mm_W1.6mm_P2.50mm, F.Cu at (60.7, 41.1)
- added ADR0_U0: ~, Package_DIP:DIP-16_W7.62mm, F.Cu at (17.6, 152.8)
- added ADR0_U0_C1: 100nF, Capacitor_THT:C_Disc_D3.0mm_W1.6mm_P2.50mm, F.Cu at (69.5, 152.3)
- added ADR0_U1: ~, Package_DIP:DIP-16_W7.62mm, F.Cu at (28.4, 152.8)
- added ADR0_U1_C1: 100nF, Capacitor_THT:C_Disc_D3.0mm_W1.6mm_P2.50mm, F.Cu at (69.5, 155.5)
- added ADR1_U0: ~, Package_DIP:DIP-16_W7.62mm, F.Cu at (17.6, 59.8)
- added ADR1_U0_C1: 100 nF, Capacitor_THT:C_Disc_D3.0mm_W1.6mm_P2.50mm, F.Cu at (36.0, 81.2)
- added ADR1_U1: ~, Package_DIP:DIP-16_W7.62mm, F.Cu at (28.4, 59.8)
- added ADR1_U1_C1: 100 nF, Capacitor_THT:C_Disc_D3.0mm_W1.6mm_P2.50mm, F.Cu at (36.0, 84.3)
- added ADR2_U0: ~, Package_DIP:DIP-16_W7.62mm, F.Cu at (39.1, 59.8)
- added ADR2_U0_C1: 100 nF, Capacitor_THT:C_Disc_D3.0mm_W1.6mm_P2.50mm, F.Cu at (36.0, 87.5)
- added ADR2_U1: ~, Package_DIP:DIP-16_W7.62mm, F.Cu at (49.9, 59.8)
- added ADR2_U1_C1: 100 nF, Capacitor_THT:C_Disc_D3.0mm_W1.6mm_P2.50mm, F.Cu at (36.0, 90.6)
- added ALUMUX_U0: 74HC151, Package_DIP:DIP-16_W7.62mm, F.Cu at (39.1, 16.5)
- added ALUMUX_U0_C1: 100 nF, Capacitor_THT:C_Disc_D3.0mm_W1.6mm_P2.50mm, F.Cu at (60.7, 44.2)
- added ALUMUX_U1: 74HC151, Package_DIP:DIP-16_W7.62mm, F.Cu at (49.9, 16.5)
- added ALUMUX_U1_C1: 100 nF, Capacitor_THT:C_Disc_D3.0mm_W1.6mm_P2.50mm, F.Cu at (60.7, 47.4)
- added ALUMUX_U2: 74HC151, Package_DIP:DIP-16_W7.62mm, F.Cu at (60.7, 16.5)
- added ALUMUX_U2_C1: 100 nF, Capacitor_THT:C_Disc_D3.0mm_W1.6mm_P2.50mm, F.Cu at (60.7, 50.5)
- added ALUMUX_U3: 74HC151, Package_DIP:DIP-16_W7.62mm, F.Cu at (71.5, 16.5)
- added ALUMUX_U3_C1: 100 nF, Capacitor_THT:C_Disc_D3.0mm_W1.6mm_P2.50mm, F.Cu at (60.7, 53.7)
- added ALUMUX_U4: 74HC151, Package_DIP:DIP-16_W7.62mm, F.Cu at (82.3, 16.5)
- added ALUMUX_U4_C1: 100 nF, Capacitor_THT:C_Disc_D3.0mm_W1.6mm_P2.50mm, F.Cu at (66.3, 37.9)
- added ALUMUX_U5: 74HC151, Package_DIP:DIP-16_W7.62mm, F.Cu at (93.0, 16.5)
- added ALUMUX_U5_C1: 100 nF, Capacitor_THT:C_Disc_D3.0mm_W1.6mm_P2.50mm, F.Cu at (66.3, 41.1)
- added ALUMUX_U6: 74HC151, Package_DIP:DIP-16_W7.62mm, F.Cu at (103.8, 16.5)
- added ALUMUX_U6_C1: 100 nF, Capacitor_THT:C_Disc_D3.0mm_W1.6mm_P2.50mm, F.Cu at (66.3, 44.2)
- added ALUMUX_U7: 74HC151, Package_DIP:DIP-16_W7.62mm, F.Cu at (114.6, 16.5)
- added ALUMUX_U7_C1: 100 nF, Capacitor_THT:C_Disc_D3.0mm_W1.6mm_P2.50mm, F.Cu at (66.3, 47.4)
- added ALU_C1: 12uF, Capacitor_THT:C_Radial_D5.0mm_H5.0mm_P2.00mm, F.Cu at (72.2, 127.1)
- added AUX_U0: 74HC273, Package_DIP:DIP-20_W7.62mm, F.Cu at (17.6, 125.8)
- added AUX_U0_C1: 100nF, Capacitor_THT:C_Disc_D3.0mm_W1.6mm_P2.50mm, F.Cu at (69.5, 158.6)
- added AUX_U1: 74HC245, Package_DIP:DIP-20_W7.62mm, F.Cu at (28.4, 125.8)
- added AUX_U1_C1: 100nF, Capacitor_THT:C_Disc_D3.0mm_W1.6mm_P2.50mm, F.Cu at (69.5, 161.8)
- added CLKINVERTER_U1: 74HC04, Package_DIP:DIP-14_W7.62mm, F.Cu at (148.9, 59.8)
- added CLKINVERTER_U_C1: 100 nF, Capacitor_THT:C_Disc_D3.0mm_W1.6mm_P2.50mm, F.Cu at (159.7, 59.3)
- added CLK_U1: LM555xN, Package_DIP:DIP-8_W7.62mm, F.Cu at (159.7, 72.4)
- added CLK_U_C1: C, Capacitor_THT:C_Disc_D3.0mm_W1.6mm_P2.50mm, F.Cu at (159.7, 62.4)
- added CLK_U_C2: 100 nF, Capacitor_THT:C_Disc_D3.0mm_W1.6mm_P2.50mm, F.Cu at (159.7, 65.6)
- added CLK_U_C3: C, Capacitor_THT:C_Disc_D3.0mm_W1.6mm_P2.50mm, F.Cu at (159.7, 68.7)
- added CLK_U_R1: R, Resistor_THT:R_Axial_DIN0204_L3.6mm_D1.6mm_P5.08mm_Horizontal, F.Cu at (148.8, 78.6)
- added COMP_U0: 74HC85, Package_DIP:DIP-16_W7.62mm, F.Cu at (125.4, 16.5)
- added COMP_U0_C1: 100 nF, Capacitor_THT:C_Disc_D3.0mm_W1.6mm_P2.50mm, F.Cu at (66.3, 50.5)
- added COMP_U0_C2: 100 nF, Capacitor_THT:C_Disc_D3.0mm_W1.6mm_P2.50mm, F.Cu at (66.3, 53.7)
- added COMP_U1: 74HC85, Package_DIP:DIP-16_W7.62mm, F.Cu at (136.2, 16.5)
- added CU_C1: 12uF, Capacitor_THT:C_Radial_D5.0mm_H5.0mm_P2.00mm, F.Cu at (72.2, 133.6)
- added DECODER_U0: 28C64, Package_DIP:DIP-28_W15.24mm, F.Cu at (80.0, 125.9)
- added DECODER_U0_C1: 100 nF, Capacitor_THT:C_Disc_D3.0mm_W1.6mm_P2.50mm, F.Cu at (80.0, 162.5)
- added DECODER_U1: 28C64, Package_DIP:DIP-28_W15.24mm, F.Cu at (98.4, 125.9)
- added DECODER_U1_C1: 100 nF, Capacitor_THT:C_Disc_D3.0mm_W1.6mm_P2.50mm, F.Cu at (80.0, 165.7)
- added DECODER_U2: 28C64, Package_DIP:DIP-28_W15.24mm, F.Cu at (116.8, 125.9)
- added DECODER_U2_C1: 100 nF, Capacitor_THT:C_Disc_D3.0mm_W1.6mm_P2.50mm, F.Cu at (80.0, 168.8)
- added DTA_U1: 74HC273, Package_DIP:DIP-20_W7.62mm, F.Cu at (39.1, 125.8)
- added DTA_U_C1: 100nF, Capacitor_THT:C_Disc_D3.0mm_W1.6mm_P2.50mm, F.Cu at (69.5, 164.9)
- added DTB_U1: 74HC273, Package_DIP:DIP-20_W7.62mm, F.Cu at (49.9, 125.8)
- added DTB_U_C1: 100nF, Capacitor_THT:C_Disc_D3.0mm_W1.6mm_P2.50mm, F.Cu at (69.5, 168.1)
- added IC_U1: ~, Package_DIP:DIP-16_W7.62mm, F.Cu at (39.1, 152.8)
- added IC_U_C1: 100nF, Capacitor_THT:C_Disc_D3.0mm_W1.6mm_P2.50mm, F.Cu at (69.5, 171.2)
- added INPFLAG_U1: 74HC245, Package_DIP:DIP-20_W7.62mm, F.Cu at (137.2, 125.8)
- added INPFLAG_U_C1: 100 nF, Capacitor_THT:C_Disc_D3.0mm_W1.6mm_P2.50mm, F.Cu at (157.2, 152.3)
- added INP_CONN0: Conn_01x02, Connector_PinHeader_2.54mm:PinHeader_1x02_P2.54mm_Vertical, F.Cu at (163.5, 153.0)
- added INP_CONN1: Conn_01x02, Connector_PinHeader_2.54mm:PinHeader_1x02_P2.54mm_Vertical, F.Cu at (168.1, 153.0)
- added INP_CONN2: Conn_01x08, Connector_PinHeader_2.54mm:PinHeader_1x08_P2.54mm_Vertical, F.Cu at (137.9, 153.0)
- added INP_U0: 74HC273, Package_DIP:DIP-20_W7.62mm, F.Cu at (148.0, 125.8)
- added INP_U0_C1: 100 nF, Capacitor_THT:C_Disc_D3.0mm_W1.6mm_P2.50mm, F.Cu at (157.2, 155.5)
- added INP_U1: 74HC245, Package_DIP:DIP-20_W7.62mm, F.Cu at (158.8, 125.8)
- added INP_U1_C1: 100 nF, Capacitor_THT:C_Disc_D3.0mm_W1.6mm_P2.50mm, F.Cu at (157.2, 158.6)
- added IODFLIPFLOP_U1: 74HC74, Package_DIP:DIP-14_W7.62mm, F.Cu at (146.4, 152.8)
- added IODFLIPFLOP_U_C1: 100 nF, Capacitor_THT:C_Disc_D3.0mm_W1.6mm_P2.50mm, F.Cu at (157.2, 161.8)
- added IR_U1: 74HC273, Package_DIP:DIP-20_W7.62mm, F.Cu at (60.7, 125.8)
- added IR_U_C1: 100 nF, Capacitor_THT:C_Disc_D3.0mm_W1.6mm_P2.50mm, F.Cu at (69.5, 174.4)
- added NAND_U0: 74HC00, Package_DIP:DIP-14_W7.62mm, F.Cu at (17.6, 38.4)
- added NAND_U0_C1: 100 nF, Capacitor_THT:C_Disc_D3.0mm_W1.6mm_P2.50mm, F.Cu at (72.0, 37.9)
- added NAND_U1: 74HC00, Package_DIP:DIP-14_W7.62mm, F.Cu at (28.4, 38.4)
- added NAND_U1_C1: 100 nF, Capacitor_THT:C_Disc_D3.0mm_W1.6mm_P2.50mm, F.Cu at (72.0, 41.1)
- added OUT_CONN0: Conn_01x02, Connector_PinHeader_2.54mm:PinHeader_1x02_P2.54mm_Vertical, F.Cu at (172.7, 153.0)
- added OUT_CONN1: Conn_01x01, Connector_PinHeader_2.54mm:PinHeader_1x01_P2.54mm_Vertical, F.Cu at (177.3, 153.0)
- added OUT_CONN2: Conn_01x08, Connector_PinHeader_2.54mm:PinHeader_1x08_P2.54mm_Vertical, F.Cu at (142.5, 153.0)
- added OUT_FLAG_U1: 74HC245, Package_DIP:DIP-20_W7.62mm, F.Cu at (169.5, 125.8)
- added OUT_FLAG_U_C1: 100 nF, Capacitor_THT:C_Disc_D3.0mm_W1.6mm_P2.50mm, F.Cu at (157.2, 164.9)
- added OUT_U1: 74HC273, Package_DIP:DIP-20_W7.62mm, F.Cu at (180.3, 125.8)
- added OUT_U_C1: 100 nF, Capacitor_THT:C_Disc_D3.0mm_W1.6mm_P2.50mm, F.Cu at (157.2, 168.1)
- added PC_U0: ~, Package_DIP:DIP-16_W7.62mm, F.Cu at (60.7, 59.8)
- added PC_U0_C1: 100 nF, Capacitor_THT:C_Disc_D3.0mm_W1.6mm_P2.50mm, F.Cu at (36.0, 93.8)
- added PC_U1: ~, Package_DIP:DIP-16_W7.62mm, F.Cu at (71.5, 59.8)
- added PC_U1_C1: 100 nF, Capacitor_THT:C_Disc_D3.0mm_W1.6mm_P2.50mm, F.Cu at (36.0, 96.9)
- added PC_U2: ~, Package_DIP:DIP-16_W7.62mm, F.Cu at (82.3, 59.8)
- added PC_U2_C1: 100 nF, Capacitor_THT:C_Disc_D3.0mm_W1.6mm_P2.50mm, F.Cu at (36.0, 100.1)
- added PC_U3: ~, Package_DIP:DIP-16_W7.62mm, F.Cu at (93.0, 59.8)
- added PC_U3_C1: 100 nF, Capacitor_THT:C_Disc_D3.0mm_W1.6mm_P2.50mm, F.Cu at (41.6, 81.2)
- added RAM_C1: 12uF, Capacitor_THT:C_Radial_D5.0mm_H5.0mm_P2.00mm, F.Cu at (72.2, 140.2)
- added RAM_U1: ~, Package_DIP:DIP-24_18.0mmx34.29mm_W15.24mm, F.Cu at (50.5, 154.7)
- added RAM_U_C1: 100nF, Capacitor_THT:C_Disc_D3.0mm_W1.6mm_P2.50mm, F.Cu at (69.5, 177.5)
- added ROMMUX_U0: ~, Package_DIP:DIP-16_W7.62mm, F.Cu at (103.8, 59.8)
- added ROMMUX_U0_C1: 100 nF, Capacitor_THT:C_Disc_D3.0mm_W1.6mm_P2.50mm, F.Cu at (41.6, 84.3)
- added ROMMUX_U1: ~, Package_DIP:DIP-16_W7.62mm, F.Cu at (114.6, 59.8)
- added ROMMUX_U1_C1: 100 nF, Capacitor_THT:C_Disc_D3.0mm_W1.6mm_P2.50mm, F.Cu at (41.6, 87.5)
- added ROMMUX_U2: ~, Package_DIP:DIP-16_W7.62mm, F.Cu at (125.4, 59.8)
- added ROMMUX_U2_C1: 100 nF, Capacitor_THT:C_Disc_D3.0mm_W1.6mm_P2.50mm, F.Cu at (41.6, 90.6)
- added ROMMUX_U3: ~, Package_DIP:DIP-16_W7.62mm, F.Cu at (136.2, 59.8)
- added ROMMUX_U3_C1: 100 nF, Capacitor_THT:C_Disc_D3.0mm_W1.6mm_P2.50mm, F.Cu at (41.6, 93.8)
- added ROM_C1: 12uF, Capacitor_THT:C_Radial_D5.0mm_H5.0mm_P2.00mm, F.Cu at (72.2, 146.7)
- added ROM_U1: 28C512, Package_DIP:DIP-32_W15.24mm, F.Cu at (17.6, 81.6)
- added ROM_U_C1: 100 nF, Capacitor_THT:C_Disc_D3.0mm_W1.6mm_P2.50mm, F.Cu at (41.6, 96.9)
- added SWT_U1: 74HC74, Package_DIP:DIP-14_W7.62mm, F.Cu at (36.0, 103.7)
- added SWT_U_C1: 100 nF, Capacitor_THT:C_Disc_D3.0mm_W1.6mm_P2.50mm, F.Cu at (41.6, 100.1)
- added USB_CONN1: USB_C_Receptacle_PowerOnly_6P, Connector_USB:USB_C_Receptacle_GCT_USB4125-xx-x-0190_6P_TopMnt_Horizontal, F.Cu at (21.9, 177.5)
- added USB_CONN_C1: 1nF >=50V, Capacitor_THT:C_Disc_D3.0mm_W1.6mm_P2.50mm, F.Cu at (69.5, 180.7)
- added USB_CONN_R1: 5.1k, Resistor_THT:R_Axial_DIN0204_L3.6mm_D1.6mm_P5.08mm_Horizontal, F.Cu at (17.5, 183.5)
- added XOR_U0: 74HC86, Package_DIP:DIP-14_W7.62mm, F.Cu at (39.1, 38.4)
- added XOR_U0_C1: 100 nF, Capacitor_THT:C_Disc_D3.0mm_W1.6mm_P2.50mm, F.Cu at (72.0, 44.2)
- added XOR_U1: 74HC86, Package_DIP:DIP-14_W7.62mm, F.Cu at (49.9, 38.4)
- added XOR_U1_C1: 100 nF, Capacitor_THT:C_Disc_D3.0mm_W1.6mm_P2.50mm, F.Cu at (72.0, 47.4)
